Commit message: New Creatures

File: body.urdf (robot description, URDF)
Before this commit: robot robot, 9 links, 8 joints
Links:
- link FLT: geometry collision box size=0.15 0.15 0.75; visual box size=0.15 0.15 0.75
- link FRT: geometry collision box size=0.15 0.15 0.75; visual box size=0.15 0.15 0.75
- link Torso: geometry collision box size=1 0.5 0.5; visual box size=1 0.5 0.5
Joints:
- joint Torso_BLT: origin xyz=-1 -0.5 1.25 rpy=0 0 0 -> xyz=.425 0.1775 1 rpy=0 0 0
- joint Torso_BRT: origin xyz=-1 0.5 1.25 rpy=0 0 0 -> xyz=.425 -0.1775 1 rpy=0 0 0
- joint Torso_FLT: origin xyz=1 -0.5 1.25 rpy=0 0 0 -> xyz=-.425 0.1775 0.875 rpy=0 0 0
- joint Torso_FRT: origin xyz=1 0.5 1.25 rpy=0 0 0 -> xyz=-.425 -0.1775 0.875 rpy=0 0 0

Commit message: e

File: body.urdf (robot description, URDF)
Before this commit: robot robot, 9 links, 8 joints
Links:
- link FLT: geometry collision box size=0.15 0.15 0.5; visual box size=0.15 0.15 0.5
- link FRT: geometry collision box size=0.15 0.15 0.5; visual box size=0.15 0.15 0.5
- link Torso: geometry collision box size=2.5 2.5 1; visual box size=2.5 2.5 1
Joints:
- joint Torso_BLT: origin xyz=.425 0.1775 1 rpy=0 0 0 -> xyz=-1.25 -1.25 1.25 rpy=0 0 0
- joint Torso_BRT: origin xyz=.425 -0.1775 1 rpy=0 0 0 -> xyz=-1.25 1.25 1.25 rpy=0 0 0
- joint Torso_FLT: origin xyz=-.425 0.1775 0.875 rpy=0 0 0 -> xyz=1.25 0 1.25 rpy=0 0 0
- joint Torso_FRT: origin xyz=-.425 -0.1775 0.875 rpy=0 0 0 -> xyz=-1.25 0 1.25 rpy=0 0 0
